File: opip2e_fan.kicad_pcb (KiCad board)
At the start: 2 copper layers, 22.4 x 53.3 mm, 10 parts, among them J1 Conn_02x20_Odd_Even, J2 Conn_01x02_Male, Q1 Q_NPN_CBE, U1 ATtiny25-20PU

Commit message: improved pads/vias
Parts:
- moved D1 1.98 mm to (106.2, 77.7), turned to 180 degrees
- moved J2 0.76 mm to (102.9, 75.2)
- moved R3 0.26 mm to (96.8, 66.0)
- moved D3 0.25 mm to (97.8, 71.9)
- moved R2 0.25 mm to (99.1, 66.0)
- moved D4 0.25 mm to (97.8, 77.0)
Routing:
- net +5V: track 38.8 -> 40.5 mm
- net I2C_SCL: track 24.9 -> 24.2 mm
- net Net-(D4-Pad2): track 9.35 -> 9.87 mm
Other:
- net class Default: via_dia 0.8 -> 0.5; via_drill 0.4 -> 0.3
- net class power: via_dia 0.8 -> 0.5; via_drill 0.4 -> 0.3
